Commit message: add gripper grasp point to srdf

File: srdf/ur_macro.srdf.xacro (robot description, xacro)
@@ -11,7 +11,37 @@
     <!--CHAINS - When a chain is specified, all the links along the chain (including endpoints) are included in the group. Additionally, all the joints that are parents to included links are also included. This means that joints along the chain and the parent joint of the base link are included in the group-->
     <!--SUBGROUPS - Groups can also be formed by referencing to already defined group names-->
-    <group name="${prefix}${name}_manipulator">
-      <chain base_link="${prefix}base_link" tip_link="${prefix}tool0" />
-    </group>
+    <xacro:if value="${with_gripper}">
+        <group name="${prefix}${name}_manipulator_gripper">
+            <chain base_link="${prefix}base_link" tip_link="${prefix}robotiq_grasp_point" />
+        </group>
+        <group_state name="${prefix}home" group="${prefix}${name}_manipulator_gripper">
+            <joint name="${prefix}elbow_joint" value="0" />
+            <joint name="${prefix}shoulder_lift_joint" value="-1.5707" />
+            <joint name="${prefix}shoulder_pan_joint" value="0" />
+            <joint name="${prefix}wrist_1_joint" value="0" />
+            <joint name="${prefix}wrist_2_joint" value="0" />
+            <joint name="${prefix}wrist_3_joint" value="0" />
+          </group_state>
+          <group_state name="${prefix}up" group="${prefix}${name}_manipulator_gripper">
+            <joint name="${prefix}elbow_joint" value="0" />
+            <joint name="${prefix}shoulder_lift_joint" value="-1.5707" />
+            <joint name="${prefix}shoulder_pan_joint" value="0" />
+            <joint name="${prefix}wrist_1_joint" value="-1.5707" />
+            <joint name="${prefix}wrist_2_joint" value="0" />
+            <joint name="${prefix}wrist_3_joint" value="0" />
+          </group_state>
+          <group_state name="${prefix}test_configuration" group="${prefix}${name}_manipulator_gripper">
+            <joint name="${prefix}elbow_joint" value="1.4" />
+            <joint name="${prefix}shoulder_lift_joint" value="-1.62" />
+            <joint name="${prefix}shoulder_pan_joint" value="1.54" />
+            <joint name="${prefix}wrist_1_joint" value="-1.2" />
+            <joint name="${prefix}wrist_2_joint" value="-1.6" />
+            <joint name="${prefix}wrist_3_joint" value="-0.11" />
+          </group_state>
+    </xacro:if>
+    <xacro:unless value="${with_gripper}">
+        <group name="${prefix}${name}_manipulator">
+        <chain base_link="${prefix}base_link" tip_link="${prefix}tool0" />
+        </group>
     <!--GROUP STATES - Purpose - Define a named state for a particular group, in terms of joint values. This is useful to define states like 'folded arms'-->
     <group_state name="${prefix}home" group="${prefix}${name}_manipulator">
@@ -39,4 +69,5 @@
       <joint name="${prefix}wrist_3_joint" value="-0.11" />
     </group_state>
+    </xacro:unless>
     <!--END EFFECTOR - Purpose - Represent information about an end effector.-->
     <!--VIRTUAL JOINT - Purpose - this element defines a virtual joint between a robot link and an external frame of reference (considered fixed with respect to the robot)-->

Commit message: update config files for gripper

File: srdf/ur_macro.srdf.xacro (robot description, xacro)
@@ -42,31 +42,31 @@
     <xacro:unless value="${with_gripper}">
         <group name="${prefix}${name}_manipulator">
-        <chain base_link="${prefix}base_link" tip_link="${prefix}tool0" />
+            <chain base_link="${prefix}base_link" tip_link="${prefix}tool0" />
         </group>
-    <!--GROUP STATES - Purpose - Define a named state for a particular group, in terms of joint values. This is useful to define states like 'folded arms'-->
-    <group_state name="${prefix}home" group="${prefix}${name}_manipulator">
-      <joint name="${prefix}elbow_joint" value="0" />
-      <joint name="${prefix}shoulder_lift_joint" value="-1.5707" />
-      <joint name="${prefix}shoulder_pan_joint" value="0" />
-      <joint name="${prefix}wrist_1_joint" value="0" />
-      <joint name="${prefix}wrist_2_joint" value="0" />
-      <joint name="${prefix}wrist_3_joint" value="0" />
-    </group_state>
-    <group_state name="${prefix}up" group="${prefix}${name}_manipulator">
-      <joint name="${prefix}elbow_joint" value="0" />
-      <joint name="${prefix}shoulder_lift_joint" value="-1.5707" />
-      <joint name="${prefix}shoulder_pan_joint" value="0" />
-      <joint name="${prefix}wrist_1_joint" value="-1.5707" />
-      <joint name="${prefix}wrist_2_joint" value="0" />
-      <joint name="${prefix}wrist_3_joint" value="0" />
-    </group_state>
-    <group_state name="${prefix}test_configuration" group="${prefix}${name}_manipulator">
-      <joint name="${prefix}elbow_joint" value="1.4" />
-      <joint name="${prefix}shoulder_lift_joint" value="-1.62" />
-      <joint name="${prefix}shoulder_pan_joint" value="1.54" />
-      <joint name="${prefix}wrist_1_joint" value="-1.2" />
-      <joint name="${prefix}wrist_2_joint" value="-1.6" />
-      <joint name="${prefix}wrist_3_joint" value="-0.11" />
-    </group_state>
+        <!--GROUP STATES - Purpose - Define a named state for a particular group, in terms of joint values. This is useful to define states like 'folded arms'-->
+        <group_state name="${prefix}home" group="${prefix}${name}_manipulator">
+            <joint name="${prefix}elbow_joint" value="0" />
+            <joint name="${prefix}shoulder_lift_joint" value="-1.5707" />
+            <joint name="${prefix}shoulder_pan_joint" value="0" />
+            <joint name="${prefix}wrist_1_joint" value="0" />
+            <joint name="${prefix}wrist_2_joint" value="0" />
+        <joint name="${prefix}wrist_3_joint" value="0" />
+        </group_state>
+        <group_state name="${prefix}up" group="${prefix}${name}_manipulator">
+            <joint name="${prefix}elbow_joint" value="0" />
+            <joint name="${prefix}shoulder_lift_joint" value="-1.5707" />
+            <joint name="${prefix}shoulder_pan_joint" value="0" />
+            <joint name="${prefix}wrist_1_joint" value="-1.5707" />
+            <joint name="${prefix}wrist_2_joint" value="0" />
+            <joint name="${prefix}wrist_3_joint" value="0" />
+        </group_state>
+        <group_state name="${prefix}test_configuration" group="${prefix}${name}_manipulator">
+            <joint name="${prefix}elbow_joint" value="1.4" />
+            <joint name="${prefix}shoulder_lift_joint" value="-1.62" />
+            <joint name="${prefix}shoulder_pan_joint" value="1.54" />
+            <joint name="${prefix}wrist_1_joint" value="-1.2" />
+            <joint name="${prefix}wrist_2_joint" value="-1.6" />
+            <joint name="${prefix}wrist_3_joint" value="-0.11" />
+        </group_state>
     </xacro:unless>
     <!--END EFFECTOR - Purpose - Represent information about an end effector.-->
@@ -86,10 +86,10 @@
     <xacro:if value="${with_gripper}">
         <disable_collisions link1="${prefix}wrist_3_link" link2="${prefix}robotiq_85_base_link" reason="Adjacent" />
-        <disable_collisions link1="robotiq_85_base_link" link2="robotiq_85_left_finger_link" reason="Never"/>
-        <disable_collisions link1="robotiq_85_base_link" link2="robotiq_85_left_finger_tip_link" reason="Never"/>
+        <disable_collisions link1="robotiq_85_base_link" link2="robotiq_85_left_finger_link" reason="Adjacent"/>
+        <disable_collisions link1="robotiq_85_base_link" link2="robotiq_85_left_finger_tip_link" reason="Adjacent"/>
         <disable_collisions link1="robotiq_85_base_link" link2="robotiq_85_left_inner_knuckle_link" reason="Adjacent"/>
         <disable_collisions link1="robotiq_85_base_link" link2="robotiq_85_left_knuckle_link" reason="Adjacent"/>
-        <disable_collisions link1="robotiq_85_base_link" link2="robotiq_85_right_finger_link" reason="Never"/>
-        <disable_collisions link1="robotiq_85_base_link" link2="robotiq_85_right_finger_tip_link" reason="Never"/>
+        <disable_collisions link1="robotiq_85_base_link" link2="robotiq_85_right_finger_link" reason="Adjacent"/>
+        <disable_collisions link1="robotiq_85_base_link" link2="robotiq_85_right_finger_tip_link" reason="Adjacent"/>
         <disable_collisions link1="robotiq_85_base_link" link2="robotiq_85_right_inner_knuckle_link" reason="Adjacent"/>
         <disable_collisions link1="robotiq_85_base_link" link2="robotiq_85_right_knuckle_link" reason="Adjacent"/>
@@ -97,29 +97,35 @@
         <disable_collisions link1="robotiq_85_left_finger_link" link2="robotiq_85_left_inner_knuckle_link" reason="Never"/>
         <disable_collisions link1="robotiq_85_left_finger_link" link2="robotiq_85_left_knuckle_link" reason="Adjacent"/>
-        <disable_collisions link1="robotiq_85_left_finger_link" link2="robotiq_85_right_finger_link" reason="Never"/>
-        <disable_collisions link1="robotiq_85_left_finger_link" link2="robotiq_85_right_finger_tip_link" reason="Never"/>
-        <disable_collisions link1="robotiq_85_left_finger_link" link2="robotiq_85_right_inner_knuckle_link" reason="Never"/>
-        <disable_collisions link1="robotiq_85_left_finger_link" link2="robotiq_85_right_knuckle_link" reason="Never"/>
+        <disable_collisions link1="robotiq_85_left_finger_link" link2="robotiq_85_right_finger_link" reason="Adjacent"/>
+        <disable_collisions link1="robotiq_85_left_finger_link" link2="robotiq_85_right_finger_tip_link" reason="Adjacent"/>
+        <disable_collisions link1="robotiq_85_left_finger_link" link2="robotiq_85_right_inner_knuckle_link" reason="Adjacent"/>
+        <disable_collisions link1="robotiq_85_left_finger_link" link2="robotiq_85_right_knuckle_link" reason="Adjacent"/>
         <disable_collisions link1="robotiq_85_left_finger_tip_link" link2="robotiq_85_left_inner_knuckle_link" reason="Default"/>
-        <disable_collisions link1="robotiq_85_left_finger_tip_link" link2="robotiq_85_left_knuckle_link" reason="Never"/>
-        <disable_collisions link1="robotiq_85_left_finger_tip_link" link2="robotiq_85_right_finger_link" reason="Never"/>
-        <disable_collisions link1="robotiq_85_left_finger_tip_link" link2="robotiq_85_right_finger_tip_link" reason="Never"/>
-        <disable_collisions link1="robotiq_85_left_finger_tip_link" link2="robotiq_85_right_inner_knuckle_link" reason="Never"/>
-        <disable_collisions link1="robotiq_85_left_finger_tip_link" link2="robotiq_85_right_knuckle_link" reason="Never"/>
-        <disable_collisions link1="robotiq_85_left_inner_knuckle_link" link2="robotiq_85_left_knuckle_link" reason="Never"/>
-        <disable_collisions link1="robotiq_85_left_inner_knuckle_link" link2="robotiq_85_right_finger_link" reason="Never"/>
-        <disable_collisions link1="robotiq_85_left_inner_knuckle_link" link2="robotiq_85_right_finger_tip_link" reason="Never"/>
-        <disable_collisions link1="robotiq_85_left_inner_knuckle_link" link2="robotiq_85_right_inner_knuckle_link" reason="Never"/>
-        <disable_collisions link1="robotiq_85_left_inner_knuckle_link" link2="robotiq_85_right_knuckle_link" reason="Never"/>
-        <disable_collisions link1="robotiq_85_left_knuckle_link" link2="robotiq_85_right_finger_link" reason="Never"/>
-        <disable_collisions link1="robotiq_85_left_knuckle_link" link2="robotiq_85_right_finger_tip_link" reason="Never"/>
-        <disable_collisions link1="robotiq_85_left_knuckle_link" link2="robotiq_85_right_inner_knuckle_link" reason="Never"/>
-        <disable_collisions link1="robotiq_85_left_knuckle_link" link2="robotiq_85_right_knuckle_link" reason="Never"/>
+        <disable_collisions link1="robotiq_85_left_finger_tip_link" link2="robotiq_85_left_knuckle_link" reason="Adjacent"/>
+        <disable_collisions link1="robotiq_85_left_finger_tip_link" link2="robotiq_85_right_finger_link" reason="Adjacent"/>
+        <disable_collisions link1="robotiq_85_left_finger_tip_link" link2="robotiq_85_right_finger_tip_link" reason="Adjacent"/>
+        <disable_collisions link1="robotiq_85_left_finger_tip_link" link2="robotiq_85_right_inner_knuckle_link" reason="Adjacent"/>
+        <disable_collisions link1="robotiq_85_left_finger_tip_link" link2="robotiq_85_right_knuckle_link" reason="Adjacent"/>
+        <disable_collisions link1="robotiq_85_left_inner_knuckle_link" link2="robotiq_85_left_knuckle_link" reason="Adjacent"/>
+        <disable_collisions link1="robotiq_85_left_inner_knuckle_link" link2="robotiq_85_right_finger_link" reason="Adjacent"/>
+        <disable_collisions link1="robotiq_85_left_inner_knuckle_link" link2="robotiq_85_right_finger_tip_link" reason="Adjacent"/>
+        <disable_collisions link1="robotiq_85_left_inner_knuckle_link" link2="robotiq_85_right_inner_knuckle_link" reason="Adjacent"/>
+        <disable_collisions link1="robotiq_85_left_inner_knuckle_link" link2="robotiq_85_right_knuckle_link" reason="Adjacent"/>
+        <disable_collisions link1="robotiq_85_left_knuckle_link" link2="robotiq_85_right_finger_link" reason="Adjacent"/>
+        <disable_collisions link1="robotiq_85_left_knuckle_link" link2="robotiq_85_right_finger_tip_link" reason="Adjacent"/>
+        <disable_collisions link1="robotiq_85_left_knuckle_link" link2="robotiq_85_right_inner_knuckle_link" reason="Adjacent"/>
+        <disable_collisions link1="robotiq_85_left_knuckle_link" link2="robotiq_85_right_knuckle_link" reason="Adjacent"/>
         <disable_collisions link1="robotiq_85_right_finger_link" link2="robotiq_85_right_finger_tip_link" reason="Adjacent"/>
-        <disable_collisions link1="robotiq_85_right_finger_link" link2="robotiq_85_right_inner_knuckle_link" reason="Never"/>
+        <disable_collisions link1="robotiq_85_right_finger_link" link2="robotiq_85_right_inner_knuckle_link" reason="Adjacent"/>
         <disable_collisions link1="robotiq_85_right_finger_link" link2="robotiq_85_right_knuckle_link" reason="Adjacent"/>
         <disable_collisions link1="robotiq_85_right_finger_tip_link" link2="robotiq_85_right_inner_knuckle_link" reason="Default"/>
-        <disable_collisions link1="robotiq_85_right_finger_tip_link" link2="robotiq_85_right_knuckle_link" reason="Never"/>
-        <disable_collisions link1="robotiq_85_right_inner_knuckle_link" link2="robotiq_85_right_knuckle_link" reason="Never"/>
+        <disable_collisions link1="robotiq_85_right_finger_tip_link" link2="robotiq_85_right_knuckle_link" reason="Adjacent"/>
+        <disable_collisions link1="robotiq_85_right_inner_knuckle_link" link2="robotiq_85_right_knuckle_link" reason="Adjacent"/>
+        <!-- <disable_collisions link1="${prefix}forearm_link" link2="robotiq_85_left_finger_link" reason="Never"/>
+        <disable_collisions link1="${prefix}forearm_link" link2="robotiq_85_right_finger_link" reason="Never"/>
+        <disable_collisions link1="${prefix}forearm_link" link2="robotiq_85_right_finger_tip_link" reason="Never"/>
+        <disable_collisions link1="${prefix}forearm_link" link2="robotiq_85_left_finger_tip_link" reason="Never"/>
+        <disable_collisions link1="${prefix}forearm_link" link2="robotiq_85_left_knuckle_link" reason="Never"/>
+        <disable_collisions link1="${prefix}forearm_link" link2="robotiq_85_right_knuckle_link" reason="Never"/> -->
     </xacro:if>
   </xacro:macro>
