Commit message: update srdf for gripper grasp point control

File: srdf/ur_macro.srdf.xacro (robot description, xacro)
@@ -11,15 +11,14 @@
     <!--CHAINS - When a chain is specified, all the links along the chain (including endpoints) are included in the group. Additionally, all the joints that are parents to included links are also included. This means that joints along the chain and the parent joint of the base link are included in the group-->
     <!--SUBGROUPS - Groups can also be formed by referencing to already defined group names-->
-    <xacro:if value="${with_gripper}">
-        <group name="${prefix}${gripper_name}">
-          <joint name="${prefix}${gripper_name}_gripper_base_joint"/>
-          <joint name="${prefix}${gripper_name}_r_finger_joint"/>
-          <joint name="${prefix}${gripper_name}_l_finger_joint"/>
-          <joint name="${prefix}${gripper_name}_grasp_point"/>
-        </group>
-    </xacro:if>
-        <group name="${prefix}${name}_manipulator">
-            <chain base_link="${prefix}base_link" tip_link="${prefix}tool0" />
-        </group>
+        <xacro:if value="${with_gripper}">
+            <group name="${prefix}${name}_manipulator">
+                <chain base_link="${prefix}base_link" tip_link="${prefix}${gripper_name}_grasp_point" />
+            </group>
+        </xacro:if>
+        <xacro:unless value="${with_gripper}">
+            <group name="${prefix}${name}_manipulator">
+                <chain base_link="${prefix}base_link" tip_link="${prefix}tool0" />
+            </group>
+        </xacro:unless>
         <!--GROUP STATES - Purpose - Define a named state for a particular group, in terms of joint values. This is useful to define states like 'folded arms'-->
         <group_state name="${prefix}home" group="${prefix}${name}_manipulator">
@@ -48,7 +47,4 @@
         </group_state>
     <!--END EFFECTOR - Purpose - Represent information about an end effector.-->
-    <xacro:if value="${with_gripper}">
-      <end_effector name="${gripper_name}" parent_link="${prefix}tool0" group="${prefix}${gripper_name}"/>
-    </xacro:if>
     <!--VIRTUAL JOINT - Purpose - this element defines a virtual joint between a robot link and an external frame of reference (considered fixed with respect to the robot)-->
     <!--DISABLE COLLISIONS - By default it is assumed that any link of the robot could potentially come into collision with any other link in the robot. This tag disables collision checking between a specified pair of links. -->
@@ -69,48 +65,4 @@
       <disable_collisions link1="${gripper_name}_gripper_base_link" link2="${gripper_name}_r_finger_link" reason="Adjacent"/>
       <disable_collisions link1="${gripper_name}_r_finger_link" link2="${gripper_name}_l_finger_link" reason="Adjacent"/>
-        <!-- <disable_collisions link1="${prefix}wrist_3_link" link2="${prefix}robotiq_85_base_link" reason="Adjacent" />
-        <disable_collisions link1="robotiq_85_base_link" link2="robotiq_85_left_finger_link" reason="Adjacent"/>
-        <disable_collisions link1="robotiq_85_base_link" link2="robotiq_85_left_finger_tip_link" reason="Adjacent"/>
-        <disable_collisions link1="robotiq_85_base_link" link2="robotiq_85_left_inner_knuckle_link" reason="Adjacent"/>
-        <disable_collisions link1="robotiq_85_base_link" link2="robotiq_85_left_knuckle_link" reason="Adjacent"/>
-        <disable_collisions link1="robotiq_85_base_link" link2="robotiq_85_right_finger_link" reason="Adjacent"/>
-        <disable_collisions link1="robotiq_85_base_link" link2="robotiq_85_right_finger_tip_link" reason="Adjacent"/>
-        <disable_collisions link1="robotiq_85_base_link" link2="robotiq_85_right_inner_knuckle_link" reason="Adjacent"/>
-        <disable_collisions link1="robotiq_85_base_link" link2="robotiq_85_right_knuckle_link" reason="Adjacent"/>
-        <disable_collisions link1="robotiq_85_left_finger_link" link2="robotiq_85_left_finger_tip_link" reason="Adjacent"/>
-        <disable_collisions link1="robotiq_85_left_finger_link" link2="robotiq_85_left_inner_knuckle_link" reason="Never"/>
-        <disable_collisions link1="robotiq_85_left_finger_link" link2="robotiq_85_left_knuckle_link" reason="Adjacent"/>
-        <disable_collisions link1="robotiq_85_left_finger_link" link2="robotiq_85_right_finger_link" reason="Adjacent"/>
-        <disable_collisions link1="robotiq_85_left_finger_link" link2="robotiq_85_right_finger_tip_link" reason="Adjacent"/>
-        <disable_collisions link1="robotiq_85_left_finger_link" link2="robotiq_85_right_inner_knuckle_link" reason="Adjacent"/>
-        <disable_collisions link1="robotiq_85_left_finger_link" link2="robotiq_85_right_knuckle_link" reason="Adjacent"/>
-        <disable_collisions link1="robotiq_85_left_finger_tip_link" link2="robotiq_85_left_inner_knuckle_link" reason="Default"/>
-        <disable_collisions link1="robotiq_85_left_finger_tip_link" link2="robotiq_85_left_knuckle_link" reason="Adjacent"/>
-        <disable_collisions link1="robotiq_85_left_finger_tip_link" link2="robotiq_85_right_finger_link" reason="Adjacent"/>
-        <disable_collisions link1="robotiq_85_left_finger_tip_link" link2="robotiq_85_right_finger_tip_link" reason="Adjacent"/>
-        <disable_collisions link1="robotiq_85_left_finger_tip_link" link2="robotiq_85_right_inner_knuckle_link" reason="Adjacent"/>
-        <disable_collisions link1="robotiq_85_left_finger_tip_link" link2="robotiq_85_right_knuckle_link" reason="Adjacent"/>
-        <disable_collisions link1="robotiq_85_left_inner_knuckle_link" link2="robotiq_85_left_knuckle_link" reason="Adjacent"/>
-        <disable_collisions link1="robotiq_85_left_inner_knuckle_link" link2="robotiq_85_right_finger_link" reason="Adjacent"/>
-        <disable_collisions link1="robotiq_85_left_inner_knuckle_link" link2="robotiq_85_right_finger_tip_link" reason="Adjacent"/>
-        <disable_collisions link1="robotiq_85_left_inner_knuckle_link" link2="robotiq_85_right_inner_knuckle_link" reason="Adjacent"/>
-        <disable_collisions link1="robotiq_85_left_inner_knuckle_link" link2="robotiq_85_right_knuckle_link" reason="Adjacent"/>
-        <disable_collisions link1="robotiq_85_left_knuckle_link" link2="robotiq_85_right_finger_link" reason="Adjacent"/>
-        <disable_collisions link1="robotiq_85_left_knuckle_link" link2="robotiq_85_right_finger_tip_link" reason="Adjacent"/>
-        <disable_collisions link1="robotiq_85_left_knuckle_link" link2="robotiq_85_right_inner_knuckle_link" reason="Adjacent"/>
-        <disable_collisions link1="robotiq_85_left_knuckle_link" link2="robotiq_85_right_knuckle_link" reason="Adjacent"/>
-        <disable_collisions link1="robotiq_85_right_finger_link" link2="robotiq_85_right_finger_tip_link" reason="Adjacent"/>
-        <disable_collisions link1="robotiq_85_right_finger_link" link2="robotiq_85_right_inner_knuckle_link" reason="Adjacent"/>
-        <disable_collisions link1="robotiq_85_right_finger_link" link2="robotiq_85_right_knuckle_link" reason="Adjacent"/>
-        <disable_collisions link1="robotiq_85_right_finger_tip_link" link2="robotiq_85_right_inner_knuckle_link" reason="Default"/>
-        <disable_collisions link1="robotiq_85_right_finger_tip_link" link2="robotiq_85_right_knuckle_link" reason="Adjacent"/>
-        <disable_collisions link1="robotiq_85_right_inner_knuckle_link" link2="robotiq_85_right_knuckle_link" reason="Adjacent"/>
-        <disable_collisions link1="robotiq_85_base_link" link2="rgbd_camera" reason="Adjacent"/> -->
-        <!-- <disable_collisions link1="${prefix}forearm_link" link2="robotiq_85_left_finger_link" reason="Never"/>
-        <disable_collisions link1="${prefix}forearm_link" link2="robotiq_85_right_finger_link" reason="Never"/>
-        <disable_collisions link1="${prefix}forearm_link" link2="robotiq_85_right_finger_tip_link" reason="Never"/>
-        <disable_collisions link1="${prefix}forearm_link" link2="robotiq_85_left_finger_tip_link" reason="Never"/>
-        <disable_collisions link1="${prefix}forearm_link" link2="robotiq_85_left_knuckle_link" reason="Never"/>
-        <disable_collisions link1="${prefix}forearm_link" link2="robotiq_85_right_knuckle_link" reason="Never"/> -->
     </xacro:if>
   </xacro:macro>
